Commit message: added empty world. changed meshes for spawn_objects - now with correct normals. added pkg object_recognition - subscriber and publisher: hough lines, some example pictures

File: shakey_spawn_objects/models/box.urdf (robot description, URDF)
Before this commit: robot box_model, 1 links, 0 joints
Links:
- link box: geometry collision mesh filename=package://shakey_spawn_objects/meshes/box.stl; visual mesh filename=package://shakey_spawn_objects/meshes/box.stl

File: shakey_spawn_objects/models/wedge.urdf (robot description, URDF)
Before this commit: robot wedge_model, 1 links, 0 joints
Links:
- link wedge: geometry collision mesh filename=package://shakey_spawn_objects/meshes/wedge.stl; visual mesh filename=package://shakey_spawn_objects/meshes/wedge.stl
